Commit message: Modifications needed for PDDL benchmark domain

File: highlevel_planning_ros/data/models/container/container_no_lid.urdf.xacro (robot description, xacro)
@@ -10,5 +10,5 @@
   <inertial>
     <origin rpy="0 0 0" xyz="0 0 0"/>
-    <mass value="0.0"/>
+    <mass value="0.001"/>
     <inertia ixx="1" ixy="0" ixz="0" iyy="1" iyz="0" izz="1"/>
   </inertial>

File: highlevel_planning_ros/data/models/container/lid.urdf.xacro (robot description, xacro)
@@ -10,5 +10,5 @@
   <inertial>
     <origin rpy="0 0 0" xyz="0 0 0"/>
-    <mass value="0.1"/>
+    <mass value="0.001"/>
     <inertia ixx="1" ixy="0" ixz="0" iyy="1" iyz="0" izz="1"/>
   </inertial>

File: highlevel_planning_ros/data/models/table/table.urdf (robot description, URDF)
Before this commit: robot table.urdf, 1 links, 0 joints
Links:
- link baseLink: mass .0 -> 20.0
